File: lab1elecf/astable/astable.kicad_sch (KiCad schematic)
At the start: 7 parts, among them J1 Conn_01x02, J2 Conn_01x02, U1 ICM7555xB

Commit message: VCC Y GND
Connections:
- net GND: now reaches C1.2, C2.1, J1.2 (Pin_2), J2.2 (Pin_2), U1.1 (GND)
- net VCC: now reaches J1.1 (Pin_1), R1.1, U1.4 (R), U1.8 (VCC)
